Commit message: Add launch file to spawn firefly and firely plus load

File: rotors_simulator/rotors_description/urdf/firefly/firefly.xacro (robot description, xacro)
@@ -47,5 +47,5 @@
   </xacro:property>
   <!-- Included URDF Files -->
-  <xacro:include filename="$(find rotors_description)/urdf/multirotor_base.xacro" />
+  <xacro:include filename="$(find rotors_description)/urdf/firefly/multirotor_base.xacro" />
   <!-- Instantiate multirotor_base_macro once -->
   <xacro:multirotor_base_macro
@@ -184,85 +184,3 @@
     <xacro:insert_block name="rotor_inertia" />
   </xacro:vertical_rotor>
-  <!-- Joint bewteen quad and next joint -->
-  <joint name="pre_load_hinge" type="continuous">
-    <parent link="${namespace}/base_link"/>
-    <child link="pre_load"/>
-    <origin xyz="0 0 0" rpy="0 0 0"/>
-    <axis xyz="1 0 0"/>
-    <!--<calibration rising="0.0"/> -->
-    <!--<dynamics damping="0.0" friction="0.0"/> -->
-    <!--<limit effort="50000" lower="-1.57079632679" upper="1.57079632679" velocity="10000"/>-->
-    <!--<safety_controller k_velocity="10" k_position="15" soft_lower_limit="-2.0" soft_upper_limit="0.5" /> -->
-  </joint>
-  <!-- Load -->
-  <link name="pre_load">
-    <visual>
-      <origin xyz="0 0 0" rpy="0 0 0"/>
-      <geometry>
-        <sphere radius="0.001"/>
-      </geometry>
-      <material name="orange"/>
-    </visual>
-    <inertial>
-      <origin xyz="0 0 0" rpy="0 0 0"/>
-      <mass value="0.001"/>
-      <inertia
-       ixx="0.0001" ixy="0.0" ixz="0.0"
-       iyy="0.0001" iyz="0.0"
-       izz="0.0001"/>
-    </inertial>
-  </link>
-  <!-- Joint bewteen quad and load -->
-  <joint name="load_hinge" type="con
-    tinuous">
-    <parent link="pre_load"/>
-    <child link="load"/>
-    <origin xyz="0 0 0" rpy="0 0 0"/>
-    <axis xyz="0 1 0"/>
-    <!--<calibration rising="0.0"/> -->
-    <!--<dynamics damping="0.0" friction="0.0"/> -->
-    <!--<limit effort="50000" lower="-1.57079632679" upper="1.57079632679" velocity="10000"/>-->
-    <!--<safety_controller k_velocity="10" k_position="15" soft_lower_limit="-2.0" soft_upper_limit="0.5" /> -->
-  </joint>
-  <!-- Load -->
-  <link name="load">
-    <collision>
-      <origin xyz="0 0 -0.6" rpy="0 0 0"/>
-      <geometry>
-        <box size="0.02 0.02 0.02"/>
-      </geometry>
-    </collision>
-    <visual>
-      <origin xyz="0 0 -0.6" rpy="0 0 0"/>
-      <geometry>
-        <sphere radius="0.02"/>
-      </geometry>
-      <material name="orange"/>
-    </visual>
-    <inertial>
-      <origin xyz="0 0 -0.6" rpy="0 0 0"/>
-      <mass value="0.25"/>
-      <inertia
-       ixx="0.01" ixy="0.0" ixz="0.0"
-       iyy="0.01" iyz="0.0"
-       izz="0.01"/>
-    </inertial>
-  </link>
-  <!-- Joint bewteen quad and load -->
-  <joint name="no_load_hinge" type="fixed">
-    <parent link="load"/>
-    <child link="no_load"/>
-    <origin xyz="0 0 -0.6" rpy="0 0 0"/>
-  </joint>
-  <!-- Load -->
-  <link name="no_load">
-    <inertial>
-      <origin xyz="0 0 0" rpy="0 0 0"/>
-      <mass value="0.001"/>
-      <inertia
-       ixx="0.0001" ixy="0.0" ixz="0.0"
-       iyy="0.0001" iyz="0.0"
-       izz="0.0001"/>
-    </inertial>
-  </link>
 </robot>

File: rotors_simulator/rotors_description/urdf/firefly/firefly_base.xacro (robot description, xacro)
@@ -17,7 +17,10 @@
 -->
 <robot name="firefly" xmlns:xacro="http://ros.org/wiki/xacro">
-  <xacro:include filename="$(find rotors_description)/urdf/component_snippets.xacro" />
+  <!-- <xacro:include filename="$(find rotors_description)/urdf/component_snippets.xacro" />-->
   <!-- Instantiate firefly "mechanics" -->
-  <xacro:include filename="$(find rotors_description)/urdf/firefly.xacro" />
+  <!--<xacro:include filename="$(find rotors_description)/urdf/firefly.xacro" /> -->
+  <xacro:include filename="$(find rotors_description)/urdf/firefly/component_snippets.xacro" />
+  <!-- Instantiate firefly "mechanics" -->
+  <xacro:include filename="$(find rotors_description)/urdf/firefly/firefly.xacro" />
   <!-- Instantiate a controller. -->
   <xacro:controller_plugin_macro namespace="${namespace}" imu_sub_topic="imu" />

File: rotors_simulator/rotors_description/urdf/firefly_with_load/component_snippets_loaded.xacro (robot description, xacro)
@@ -628,9 +628,64 @@
     </xacro:imu_plugin_macro>
   </xacro:macro>
+<!-- Macro to add a generic odometry sensor. -->
+  <xacro:macro name="odometry_load_plugin_macro"
+    params="
+      namespace odometry_sensor_suffix parent_link pose_topic pose_with_covariance_topic
+      position_topic transform_topic odometry_topic parent_frame_id child_frame_id
+      mass_odometry_sensor measurement_divisor measurement_delay unknown_delay
+      noise_normal_position noise_normal_quaternion noise_normal_linear_velocity
+      noise_normal_angular_velocity noise_uniform_position
+      noise_uniform_quaternion noise_uniform_linear_velocity
+      noise_uniform_angular_velocity enable_odometry_map odometry_map
+      image_scale *inertia *origin">
+    <!-- odometry link -->
+    <link name="${namespace}/odometry_sensor${odometry_sensor_suffix}_link">
+      <inertial>
+        <xacro:insert_block name="inertia" />
+        <mass value="${mass_odometry_sensor}" />  <!-- [kg] -->
+      </inertial>
+    </link>
+    <!-- odometry joint -->
+    <joint name="${namespace}/odometry_sensor${odometry_sensor_suffix}_joint" type="revolute">
+      <parent link="${parent_link}" />
+      <!-- <xacro:insert_block name="origin" /> -->
+      <origin xyz="0 0 -0.6" rpy="0 0 0"/>
+      <child link="${namespace}/odometry_sensor${odometry_sensor_suffix}_link" />
+      <limit upper="0" lower="0" effort="0" velocity="0" />
+    </joint>
+    <gazebo>
+      <plugin filename="librotors_gazebo_odometry_plugin.so" name="odometry_sensor${odometry_sensor_suffix}">
+        <linkName>${namespace}/odometry_sensor${odometry_sensor_suffix}_link</linkName>
+        <robotNamespace>${namespace}</robotNamespace>
+        <poseTopic>${pose_topic}</poseTopic>
+        <poseWithCovarianceTopic>${pose_with_covariance_topic}</poseWithCovarianceTopic>
+        <positionTopic>${position_topic}</positionTopic>
+        <transformTopic>${transform_topic}</transformTopic>
+        <odometryTopic>${odometry_topic}</odometryTopic>
+        <parentFrameId>${parent_frame_id}</parentFrameId> <!-- Use the scoped link name here. e.g. Model::link. -->
+        <childFrameId>${child_frame_id}</childFrameId>
+        <measurementDivisor>${measurement_divisor}</measurementDivisor> <!-- only every (seq % measurementDivisor) == 0 measurement is published [int] -->
+        <measurementDelay>${measurement_delay}</measurementDelay> <!-- time that measurement gets held back before it's published in [simulation cycles (int)] -->
+        <unknownDelay>${unknown_delay}</unknownDelay> <!-- additional delay, that just gets added to the timestamp [s] -->
+        <noiseNormalPosition>${noise_normal_position}</noiseNormalPosition> <!-- standard deviation of additive white gaussian noise [m] -->
+        <noiseNormalQuaternion>${noise_normal_quaternion}</noiseNormalQuaternion> <!-- standard deviation white gaussian noise [rad]: q_m = q*quaternionFromSmallAngleApproximation(noiseNormalQ) -->
+        <noiseNormalLinearVelocity>${noise_normal_linear_velocity}</noiseNormalLinearVelocity> <!-- standard deviation of additive white gaussian noise [m/s] -->
+        <noiseNormalAngularVelocity>${noise_normal_angular_velocity}</noiseNormalAngularVelocity> <!-- standard deviation of additive white gaussian noise [rad/s] -->
+        <noiseUniformPosition>${noise_uniform_position}</noiseUniformPosition> <!-- symmetric bounds of uniform noise [m] -->
+        <noiseUniformQuaternion>${noise_uniform_quaternion}</noiseUniformQuaternion> <!-- symmetric bounds of uniform noise [rad], computation see above -->
+        <noiseUniformLinearVelocity>${noise_uniform_linear_velocity}</noiseUniformLinearVelocity> <!-- symmetric bounds of uniform noise [m/s] -->
+        <noiseUniformAngularVelocity>${noise_uniform_angular_velocity}</noiseUniformAngularVelocity> <!-- symmetric bounds of uniform noise [rad/s] -->
+        <xacro:if value="${enable_odometry_map}">
+          <covarianceImage>package://rotors_gazebo/resource/${odometry_map}</covarianceImage> <!-- a bitmap image describing where the sensor works (white), and where not (black) -->
+          <covarianceImageScale>${image_scale}</covarianceImageScale> <!-- the scale of the image in the gazebo world, if set to 1.0, 1 pixel in the image corresponds to 1 meter in the world -->
+        </xacro:if>
+      </plugin>
+    </gazebo>
+  </xacro:macro>
   <xacro:macro name="ground_truth_odometry_load" params="namespace parent_link">
     <!-- Mount a generic odometry sensor providing ground truth of LOAD. -->
     <xacro:odometry_load_plugin_macro
       namespace="${namespace}"
-      odometry_sensor_suffix="gt"
+      odometry_sensor_suffix="load"
       parent_link="${parent_link}"
       pose_topic="ground_truth/pose_load"

File: rotors_simulator/rotors_description/urdf/firefly_with_load/firefly_base_loaded.xacro (robot description, xacro)
@@ -17,7 +17,11 @@
 -->
 <robot name="firefly" xmlns:xacro="http://ros.org/wiki/xacro">
-  <xacro:include filename="$(find rotors_description)/urdf/component_snippets.xacro" />
+  <!-- <xacro:include filename="$(find rotors_description)/urdf/component_snippets.xacro" />-->
   <!-- Instantiate firefly "mechanics" -->
-  <xacro:include filename="$(find rotors_description)/urdf/firefly.xacro" />
+  <!--<xacro:include filename="$(find rotors_description)/urdf/firefly.xacro" /> -->
+  <xacro:include filename="$(find rotors_description)/urdf/firefly_with_load/component_snippets_loaded.xacro" />
+  <!-- Instantiate firefly "mechanics" -->
+  <xacro:include filename="$(find rotors_description)/urdf/firefly_with_load/firefly_loaded.xacro" />
+  <xacro:ground_truth_odometry_load namespace="${namespace}" parent_link="${namespace}/load_hinge_y" />
   <!-- Instantiate a controller. -->
   <xacro:controller_plugin_macro namespace="${namespace}" imu_sub_topic="imu" />
